Commit message: changed robot state and command interface to activate tricycle controller successfully [robot_control.xacro]

File: description/robot_control.xacro (robot description, xacro)
@@ -5,13 +5,12 @@
       <plugin>gazebo_ros2_control/GazeboSystem</plugin>
     </hardware>
-    <joint name="base_to_front_plate">
-      <command_interface name="velocity">
-        <param name="min">-10</param>
-        <param name="max">-10</param>
+    <joint name="steering_joint">
+      <command_interface name="position">
+        <param name="min">-0.5</param>
+        <param name="max">0.5</param>
       </command_interface>
-      <state_interface name="velocity"/>
       <state_interface name="position"/>
     </joint>
-    <joint name="plate_to_front_wheel">
+    <joint name="traction_joint">
       <command_interface name="velocity">
         <param name="min">-10</param>
@@ -23,7 +22,6 @@
   </ros2_control>
   <gazebo>
-    <plugin  name="gazebo_ros2_control" filename="libgazebo_ros2_control.so">
-      <parameters>
-      </parameters>
+    <plugin filename="libgazebo_ros2_control.so" name="gazebo_ros2_control">
+      <parameters>$(find Penguin)/config/my_controllers.yaml</parameters>
     </plugin>
   </gazebo>

File: description/robot_core.xacro (robot description, xacro)
@@ -126,5 +126,5 @@
     <parent link="base_link"/>
     <child link="front_plate"/>
-    <origin xyz="${chassis_length} 0 ${front_plate_height/2 + wheel_radius}"/>
+    <origin xyz="${chassis_length} 0 ${front_plate_height/2 + wheel_radius}" rpy="0 0 0"/>
     <axis xyz="0 0 1"/>
   </joint>
@@ -153,5 +153,5 @@
     <child link="front_wheel"/>
     <axis xyz="0 1 0"/>
-    <origin xyz="0 0 ${-front_plate_height/2 - wheel_radius}"/>
+    <origin xyz="0 0 ${-front_plate_height/2 - wheel_radius}" rpy="0 0 0"/>
   </joint>
   <link name="front_wheel">
