Commit message: brought back front plate to make front wheel visible in gazebo [robot_core.xacro]

File: description/my_robot.urdf.xacro (robot description, xacro)
@@ -2,3 +2,4 @@
 <robot xmlns:xacro="http://www.ros.org/wiki/xacro" name="my_robot">
   <xacro:include filename="robot_core.xacro"/>
+  <xacro:include filename="robot_control.xacro"/>
 </robot>

File: description/robot_core.xacro (robot description, xacro)
@@ -122,9 +122,36 @@
     <material>Gazebo/Blue</material>
   </gazebo>
+  <!-- FRONT PLATE -->
+   <joint name="steering_joint" type="continuous">
+    <parent link="base_link"/>
+    <child link="front_plate"/>
+    <origin xyz="${chassis_length} 0 ${front_plate_height/2 + wheel_radius}"/>
+    <axis xyz="0 0 1"/>
+  </joint>
+  <link name="front_plate">
+    <visual>
+      <geometry>
+        <cylinder radius="0.1" length="${front_plate_height}"/>
+      </geometry>
+      <origin xyz="0 0 0"/>
+      <material name="rosy_red"/>
+    </visual>
+    <collision>
+      <geometry>
+        <cylinder radius="0.1" length="${front_plate_height}"/>
+      </geometry>
+      <origin xyz="0 0 0"/>
+    </collision>
+    <xacro:inertial_cylinder mass="0.1" radius="0.1" length="${front_plate_height}"/>
+  </link>
+  <gazebo reference="front_plate">
+    <material>Gazebo/Red</material>
+  </gazebo>
   <!-- FRONT WHEEL -->
   <joint name="traction_joint" type="continuous">
-    <parent link="steer_motor"/>
+    <parent link="front_plate"/>
     <child link="front_wheel"/>
     <axis xyz="0 1 0"/>
+    <origin xyz="0 0 ${-front_plate_height/2 - wheel_radius}"/>
   </joint>
   <link name="front_wheel">
@@ -147,12 +174,4 @@
     <material>Gazebo/Yellow</material>
   </gazebo>
-  <!-- STEER MOTOR -->
-  <joint name="steering_joint" type="continuous">
-    <parent link="base_link"/>
-    <child link="steer_motor"/>
-    <origin xyz="${chassis_length} 0 0"/>
-    <axis xyz="0 0 1"/>
-  </joint>
-  <link name="steer_motor"></link>
   <!-- VACUUM HEAD -->
   <joint name="chassis_to_vacuum_head" type="fixed">

Commit message: 2D lidar added

File: description/my_robot.urdf.xacro (robot description, xacro)
@@ -1,5 +1,8 @@
 <?xml version="1.0"?>
 <robot xmlns:xacro="http://www.ros.org/wiki/xacro" name="my_robot">
+  <xacro:include filename="inertial_macro.xacro"/>
+  <xacro:include filename="property_macro.xacro"/>
   <xacro:include filename="robot_core.xacro"/>
   <xacro:include filename="robot_control.xacro"/>
+  <xacro:include filename="lidar.xacro"/>
 </robot>

File: description/robot_core.xacro (robot description, xacro)
@@ -1,26 +1,4 @@
 <?xml version="1.0"?>
 <robot xmlns:xacro="http://www.ros.org/wiki/xacro" name="my_robot">
-  <xacro:include filename="inertial_macro.xacro"/>
-  <material name="sky_blue">
-    <color rgba="0.25 0.78 1 1"/>
-  </material>
-  <material name="white">
-    <color rgba="1 1 1 1"/>
-  </material>
-  <material name="leafy_green">
-    <color rgba="0.38 0.8 0.14 1"/>
-  </material>
-  <material name="rosy_red">
-    <color rgba="0.66 0.06 0.19 1"/>
-  </material>
-  <material name="sunshine">
-    <color rgba="1 1 0 1"/>
-  </material>
-  <xacro:property name="chassis_height" value="0.2"/>
-  <xacro:property name="chassis_length" value="0.6"/>
-  <xacro:property name="chassis_width" value="0.3"/>
-  <xacro:property name="wheel_radius" value="0.1"/>
-  <xacro:property name="wheel_width" value="0.05"/>
-  <xacro:property name="front_plate_height" value="0.02"/>
   <!-- BASE LINK -->
   <link name="base_link"></link>
