Commit message: change to differential drive

File: description/inertial_macro.xacro (robot description, xacro)
@@ -17,3 +17,11 @@
     </inertial>
   </xacro:macro>
+  <xacro:macro name="inertial_sphere" params="mass radius">
+        <inertial>
+            <mass value="${mass}" />
+            <inertia ixx="${(2/5)*mass*(radius*radius)}" ixy="0.0" ixz="0.0"
+                    iyy="${(2/5)* mass*(radius*radius)}" iyz="0.0"
+                    izz="${(2/5)*mass*(radius*radius)}" />
+        </inertial>
+    </xacro:macro>
 </robot>

File: description/lidar.xacro (robot description, xacro)
@@ -31,11 +31,11 @@
         <scan>
           <horizontal>
-            <sample>360</sample>
-            <min_angle>-3.14</min_angle>
-            <max_angle>3.14</max_angle>
+            <sample>180</sample>
+            <min_angle>-1.57</min_angle>
+            <max_angle>1.57</max_angle>
           </horizontal>
         </scan>
         <range>
-          <min>0.05</min>
+          <min>0.1</min>
           <max>2</max>
         </range>

File: description/property_macro.xacro (robot description, xacro)
@@ -18,5 +18,5 @@
   <xacro:property name="chassis_height" value="0.2"/>
   <xacro:property name="chassis_length" value="0.6"/>
-  <xacro:property name="chassis_width" value="0.3"/>
+  <xacro:property name="chassis_width" value="0.6"/>
   <xacro:property name="wheel_radius" value="0.1"/>
   <xacro:property name="wheel_width" value="0.05"/>

File: description/robot_control.xacro (robot description, xacro)
@@ -5,15 +5,16 @@
       <plugin>gazebo_ros2_control/GazeboSystem</plugin>
     </hardware>
-    <joint name="steering_joint">
-      <command_interface name="position">
-        <param name="min">-1</param>
-        <param name="max">1</param>
+    <joint name="left_wheel_joint">
+      <command_interface name="velocity">
+        <param name="min">-10</param>
+        <param name="max">10</param>
       </command_interface>
+      <state_interface name="velocity"/>
       <state_interface name="position"/>
     </joint>
-    <joint name="traction_joint">
+    <joint name="right_wheel_joint">
       <command_interface name="velocity">
         <param name="min">-10</param>
-        <param name="max">-10</param>
+        <param name="max">10</param>
       </command_interface>
       <state_interface name="velocity"/>

File: description/robot_core.xacro (robot description, xacro)
@@ -5,10 +5,9 @@
   <!-- BASE FOOTPRINT -->
   <joint name="footprint_joint" type="fixed">
-    <parent name="base_link"/>
-    <child name="base_footprint"/>
+    <parent link="base_link"/>
+    <child link="base_footprint"/>
     <origin xyz="0 0 0" rpy="0 0 0"/>
   </joint>
-  <link name="base_footprint">
-  </link>
+  <link name="base_footprint"></link>
   <!-- CHASSIS -->
   <joint name="base_to_chassis" type="fixed">
@@ -29,5 +28,5 @@
       </geometry>
     </collision>
-    <xacro:inertial_box mass="2" x="${chassis_length}" y="${chassis_width}" z="${chassis_height}"/>
+    <xacro:inertial_box mass="0.7" x="${chassis_length}" y="${chassis_width}" z="${chassis_height}"/>
   </link>
   <gazebo reference="chassis">
@@ -35,8 +34,8 @@
   </gazebo>
   <!-- LEFT WHEEL -->
-  <joint name="base_link_to_left_wheel" type="continuous">
+  <joint name="left_wheel_joint" type="continuous">
     <parent link="base_link"/>
     <child link="left_wheel"/>
-    <origin xyz="0 ${-chassis_width/2} 0"/>
+    <origin xyz="${chassis_length} ${-chassis_width/2} ${wheel_radius}"/>
     <axis xyz="0 1 0"/>
   </joint>
@@ -55,5 +54,5 @@
       <origin rpy="${pi/2} 0 0"/>
     </collision>
-    <xacro:inertial_cylinder mass="0.5" radius="${wheel_radius}" length="${wheel_width}"/>
+    <xacro:inertial_cylinder mass="0.2" radius="${wheel_radius}" length="${wheel_width}"/>
   </link>
   <gazebo reference="left_wheel">
@@ -61,8 +60,8 @@
   </gazebo>
   <!-- RIGHT WHEEL -->
-  <joint name="base_link_to_right_wheel" type="continuous">
+  <joint name="right_wheel_joint" type="continuous">
     <parent link="base_link"/>
     <child link="right_wheel"/>
-    <origin xyz="0 ${chassis_width/2} 0"/>
+    <origin xyz="${chassis_length} ${chassis_width/2} ${wheel_radius}"/>
     <axis xyz="0 1 0"/>
   </joint>
@@ -81,11 +80,31 @@
       <origin rpy="${pi/2} 0 0"/>
     </collision>
-    <xacro:inertial_cylinder mass="0.5" radius="${wheel_radius}" length="${wheel_width}"/>
+    <xacro:inertial_cylinder mass="0.2" radius="${wheel_radius}" length="${wheel_width}"/>
   </link>
   <gazebo reference="right_wheel">
     <material>Gazebo/Blue</material>
   </gazebo>
+  <!-- CASTER WHEEL -->
+  <joint name="caster_wheel_joint" type="fixed">
+    <parent link="base_link"/>
+    <child link="caster_wheel"/>
+    <origin xyz="${chassis_length/3} 0 ${wheel_radius}"/>
+  </joint>
+  <link name="caster_wheel">
+    <visual>
+      <geometry>
+        <sphere radius="${wheel_radius}"/>
+      </geometry>
+      <material name="sunshine"/>
+    </visual>
+    <collision>
+      <geometry>
+        <sphere radius="${wheel_radius}"/>
+      </geometry>
+    </collision>
+    <xacro:inertial_sphere mass="0.1" radius="${wheel_radius}"/>
+  </link>
   <!-- FRONT PLATE -->
-   <joint name="steering_joint" type="continuous">
+   <!-- <joint name="steering_joint" type="continuous">
     <parent link="base_link"/>
     <child link="front_plate"/>
@@ -111,7 +130,7 @@
   <gazebo reference="front_plate">
     <material>Gazebo/Red</material>
-  </gazebo>
+  </gazebo> -->
   <!-- FRONT WHEEL -->
-  <joint name="traction_joint" type="continuous">
+  <!-- <joint name="traction_joint" type="continuous">
     <parent link="front_plate"/>
     <child link="front_wheel"/>
@@ -137,4 +156,4 @@
   <gazebo reference="front_wheel">
     <material>Gazebo/Yellow</material>
-  </gazebo>
+  </gazebo> -->
 </robot>
