Commit message: remove front_plate and joint from front_plate to front_wheel, replaced by joint from base_link to front_wheel [description/robot_core.xacro]

File: description/robot_core.xacro (robot description, xacro)
@@ -100,36 +100,10 @@
     <material>Gazebo/Blue</material>
   </gazebo>
-  <!-- FRONT HORIZONTAL PLATE -->
-  <joint name="base_to_front_plate" type="continuous">
+  <!-- FRONT WHEEL -->
+  <joint name="base_to_front_wheel" type="continuous">
     <parent link="base_link"/>
-    <child link="front_plate"/>
-    <origin xyz="${chassis_length} 0 ${front_plate_height/2 + wheel_radius}"/>
+    <child link="front_wheel"/>
+    <origin xyz="${chassis_length} 0 0"/>
     <axis xyz="0 0 1"/>
-  </joint>
-  <link name="front_plate">
-    <visual>
-      <geometry>
-        <cylinder radius="0.1" length="${front_plate_height}"/>
-      </geometry>
-      <origin xyz="0 0 0"/>
-      <material name="rosy_red"/>
-    </visual>
-    <collision>
-      <geometry>
-        <cylinder radius="0.1" length="${front_plate_height}"/>
-      </geometry>
-      <origin xyz="0 0 0"/>
-    </collision>
-    <xacro:inertial_cylinder mass="0.2" radius="0.1" length="${front_plate_height}"/>
-  </link>
-  <gazebo reference="front_plate">
-    <material>Gazebo/Red</material>
-  </gazebo>
-  <!-- FRONT WHEEL -->
-  <joint name="plate_to_front_wheel" type="continuous">
-    <parent link="front_plate"/>
-    <child link="front_wheel"/>
-    <origin xyz="0 0 ${-front_plate_height/2 - wheel_radius}"/>
-    <axis xyz="0 1 0"/>
   </joint>
   <link name="front_wheel">

Commit message: added rear axle [robot_core.xacro]

File: description/robot_core.xacro (robot description, xacro)
@@ -47,4 +47,27 @@
   <gazebo reference="chassis">
     <material>Gazebo/White</material>
+  </gazebo>
+  <!-- REAR AXLE -->
+  <joint name="base_to_rear_axle" type="fixed">
+    <parent link="base_link"/>
+    <child link="rear_axle"/>
+    <origin rpy="${pi/2} 0 0"/>
+  </joint>
+  <link name="rear_axle">
+    <visual>
+      <geometry>
+        <cylinder radius="0.01" length="${chassis_width}"/>
+      </geometry>
+      <material name="rosy_red"/>
+    </visual>
+    <collision>
+      <geometry>
+        <cylinder radius="0.01" length="${chassis_width}"/>
+      </geometry>
+    </collision>
+    <xacro:inertial_cylinder mass="0.1" radius="0.01" length="${chassis_width}"/>
+  </link>
+  <gazebo reference="rear_axle">
+    <material>Gazebo/Red</material>
   </gazebo>
   <!-- LEFT WHEEL -->

Commit message: added steering and traction joints, rear axle, fixed rear wheels [robot_core.xacro]

File: description/robot_core.xacro (robot description, xacro)
@@ -52,5 +52,4 @@
     <parent link="base_link"/>
     <child link="rear_axle"/>
-    <origin rpy="${pi/2} 0 0"/>
   </joint>
   <link name="rear_axle">
@@ -59,4 +58,5 @@
         <cylinder radius="0.01" length="${chassis_width}"/>
       </geometry>
+      <origin rpy="${pi/2} 0 0"/>
       <material name="rosy_red"/>
     </visual>
@@ -65,4 +65,5 @@
         <cylinder radius="0.01" length="${chassis_width}"/>
       </geometry>
+      <origin rpy="${pi/2} 0 0"/>
     </collision>
     <xacro:inertial_cylinder mass="0.1" radius="0.01" length="${chassis_width}"/>
@@ -72,9 +73,8 @@
   </gazebo>
   <!-- LEFT WHEEL -->
-  <joint name="base_to_left_wheel" type="continuous">
-    <parent link="base_link"/>
+  <joint name="rear_axle_to_left_wheel" type="fixed">
+    <parent link="rear_axle"/>
     <child link="left_wheel"/>
     <origin xyz="0 ${-chassis_width/2} 0"/>
-    <axis xyz="0 1 0"/>
   </joint>
   <link name="left_wheel">
@@ -98,9 +98,8 @@
   </gazebo>
   <!-- RIGHT WHEEL -->
-  <joint name="base_to_right_wheel" type="continuous">
-    <parent link="base_link"/>
+  <joint name="rear_axle_to_right_wheel" type="fixed">
+    <parent link="rear_axle"/>
     <child link="right_wheel"/>
     <origin xyz="0 ${chassis_width/2} 0"/>
-    <axis xyz="0 1 0"/>
   </joint>
   <link name="right_wheel">
@@ -124,9 +123,8 @@
   </gazebo>
   <!-- FRONT WHEEL -->
-  <joint name="base_to_front_wheel" type="continuous">
-    <parent link="base_link"/>
+  <joint name="traction_joint" type="continuous">
+    <parent link="steer_motor"/>
     <child link="front_wheel"/>
-    <origin xyz="${chassis_length} 0 0"/>
-    <axis xyz="0 0 1"/>
+    <axis xyz="0 1 0"/>
   </joint>
   <link name="front_wheel">
@@ -149,4 +147,12 @@
     <material>Gazebo/Yellow</material>
   </gazebo>
+  <!-- STEER MOTOR -->
+  <joint name="steering_joint" type="continuous">
+    <parent link="base_link"/>
+    <child link="steer_motor"/>
+    <origin xyz="${chassis_length} 0 0"/>
+    <axis xyz="0 0 1"/>
+  </joint>
+  <link name="steer_motor"></link>
   <!-- VACUUM HEAD -->
   <joint name="chassis_to_vacuum_head" type="fixed">

Commit message: removed rear axle, make the joint from base_link to rear wheels continuous, now robot can move in gazebo[robot_core.xacro]

File: description/robot_core.xacro (robot description, xacro)
@@ -48,33 +48,10 @@
     <material>Gazebo/White</material>
   </gazebo>
-  <!-- REAR AXLE -->
-  <joint name="base_to_rear_axle" type="fixed">
+  <!-- LEFT WHEEL -->
+  <joint name="base_link_to_left_wheel" type="continuous">
     <parent link="base_link"/>
-    <child link="rear_axle"/>
-  </joint>
-  <link name="rear_axle">
-    <visual>
-      <geometry>
-        <cylinder radius="0.01" length="${chassis_width}"/>
-      </geometry>
-      <origin rpy="${pi/2} 0 0"/>
-      <material name="rosy_red"/>
-    </visual>
-    <collision>
-      <geometry>
-        <cylinder radius="0.01" length="${chassis_width}"/>
-      </geometry>
-      <origin rpy="${pi/2} 0 0"/>
-    </collision>
-    <xacro:inertial_cylinder mass="0.1" radius="0.01" length="${chassis_width}"/>
-  </link>
-  <gazebo reference="rear_axle">
-    <material>Gazebo/Red</material>
-  </gazebo>
-  <!-- LEFT WHEEL -->
-  <joint name="rear_axle_to_left_wheel" type="fixed">
-    <parent link="rear_axle"/>
     <child link="left_wheel"/>
     <origin xyz="0 ${-chassis_width/2} 0"/>
+    <axis xyz="0 1 0"/>
   </joint>
   <link name="left_wheel">
@@ -98,8 +75,9 @@
   </gazebo>
   <!-- RIGHT WHEEL -->
-  <joint name="rear_axle_to_right_wheel" type="fixed">
-    <parent link="rear_axle"/>
+  <joint name="base_link_to_right_wheel" type="continuous">
+    <parent link="base_link"/>
     <child link="right_wheel"/>
     <origin xyz="0 ${chassis_width/2} 0"/>
+    <axis xyz="0 1 0"/>
   </joint>
   <link name="right_wheel">

Commit message: changed gazebo publish rate for smoother control, add some new rviz cofig files, removed vacuum_head

File: description/robot_core.xacro (robot description, xacro)
@@ -152,26 +152,3 @@
     <material>Gazebo/Yellow</material>
   </gazebo>
-  <!-- VACUUM HEAD -->
-  <joint name="chassis_to_vacuum_head" type="fixed">
-    <parent link="chassis"/>
-    <child link="vacuum_head"/>
-    <origin xyz="0 0 ${-chassis_height/2 - wheel_radius * 2 + 0.05/2}"/>
-  </joint>
-  <link name="vacuum_head">
-    <visual>
-      <geometry>
-        <box size="0.1 0.3 0.05"/>
-      </geometry>
-      <material name="leafy_green"/>
-    </visual>
-    <collision>
-      <geometry>
-        <box size="0.1 0.3 0.05"/>
-      </geometry>
-    </collision>
-    <xacro:inertial_box mass="0.1" x="0.1" y="0.3" z="0.05"/>
-  </link>
-  <gazebo reference="vacuum_head">
-    <material>Gazebo/Green</material>
-  </gazebo>
 </robot>

Commit message: robot can move backward and forward using python script now

File: description/robot_core.xacro (robot description, xacro)
@@ -110,55 +110,3 @@
     <mu2 value="0.000"/>
   </gazebo>
-  <!-- FRONT PLATE -->
-   <!-- <joint name="steering_joint" type="continuous">
-    <parent link="base_link"/>
-    <child link="front_plate"/>
-    <origin xyz="${chassis_length} 0 ${front_plate_height/2 + wheel_radius}" rpy="0 0 0"/>
-    <axis xyz="0 0 1"/>
-  </joint>
-  <link name="front_plate">
-    <visual>
-      <geometry>
-        <cylinder radius="0.1" length="${front_plate_height}"/>
-      </geometry>
-      <origin xyz="0 0 0"/>
-      <material name="rosy_red"/>
-    </visual>
-    <collision>
-      <geometry>
-        <cylinder radius="0.1" length="${front_plate_height}"/>
-      </geometry>
-      <origin xyz="0 0 0"/>
-    </collision>
-    <xacro:inertial_cylinder mass="0.1" radius="0.1" length="${front_plate_height}"/>
-  </link>
-  <gazebo reference="front_plate">
-    <material>Gazebo/Red</material>
-  </gazebo> -->
-  <!-- FRONT WHEEL -->
-  <!-- <joint name="traction_joint" type="continuous">
-    <parent link="front_plate"/>
-    <child link="front_wheel"/>
-    <axis xyz="0 1 0"/>
-    <origin xyz="0 0 ${-front_plate_height/2 - wheel_radius}" rpy="0 0 0"/>
-  </joint>
-  <link name="front_wheel">
-    <visual>
-      <geometry>
-        <cylinder radius="${wheel_radius}" length="${wheel_width}"/>
-      </geometry>
-      <origin rpy="${pi/2} 0 0"/>
-      <material name="sunshine"/>
-    </visual>
-    <collision>
-      <geometry>
-        <cylinder radius="${wheel_radius}" length="${wheel_width}"/>
-      </geometry>
-      <origin rpy="${pi/2} 0 0"/>
-    </collision>
-    <xacro:inertial_cylinder mass="0.2" radius="${wheel_radius}" length="${wheel_width}"/>
-  </link>
-  <gazebo reference="front_wheel">
-    <material>Gazebo/Yellow</material>
-  </gazebo> -->
 </robot>
