Commit message: added base footprint for slam

File: description/lidar.xacro (robot description, xacro)
@@ -38,5 +38,5 @@
         <range>
           <min>0.05</min>
-          <max>100</max>
+          <max>2</max>
         </range>
       </ray>

File: description/robot_core.xacro (robot description, xacro)
@@ -3,4 +3,12 @@
   <!-- BASE LINK -->
   <link name="base_link"></link>
+  <!-- BASE FOOTPRINT -->
+  <joint name="footprint_joint" type="fixed">
+    <parent name="base_link"/>
+    <child name="base_footprint"/>
+    <origin xyz="0 0 0" rpy="0 0 0"/>
+  </joint>
+  <link name="base_footprint">
+  </link>
   <!-- CHASSIS -->
   <joint name="base_to_chassis" type="fixed">

Commit message: map generated, added script to convert map into numpy array

File: description/lidar.xacro (robot description, xacro)
@@ -38,5 +38,5 @@
         <range>
           <min>0.1</min>
-          <max>2</max>
+          <max>10</max>
         </range>
       </ray>

File: description/robot_core.xacro (robot description, xacro)
@@ -37,5 +37,5 @@
     <parent link="base_link"/>
     <child link="left_wheel"/>
-    <origin xyz="${chassis_length} ${-chassis_width/2} ${wheel_radius}"/>
+    <origin xyz="${chassis_length/3} ${chassis_width/2} ${wheel_radius}"/>
     <axis xyz="0 1 0"/>
   </joint>
@@ -63,5 +63,5 @@
     <parent link="base_link"/>
     <child link="right_wheel"/>
-    <origin xyz="${chassis_length} ${chassis_width/2} ${wheel_radius}"/>
+    <origin xyz="${chassis_length/3} ${-chassis_width/2} ${wheel_radius}"/>
     <axis xyz="0 1 0"/>
   </joint>
@@ -89,5 +89,5 @@
     <parent link="base_link"/>
     <child link="caster_wheel"/>
-    <origin xyz="${chassis_length/3} 0 ${wheel_radius}"/>
+    <origin xyz="${3*chassis_length/4} 0 ${wheel_radius}"/>
   </joint>
   <link name="caster_wheel">
@@ -105,4 +105,9 @@
     <xacro:inertial_sphere mass="0.1" radius="${wheel_radius}"/>
   </link>
+  <gazebo reference="caster_wheel">
+    <material>Gazebo/Yellow</material>
+    <mu1 value="0.000"/>
+    <mu2 value="0.000"/>
+  </gazebo>
   <!-- FRONT PLATE -->
    <!-- <joint name="steering_joint" type="continuous">

Commit message: turn robot into a cyliner, centre wheels and base link

File: description/lidar.xacro (robot description, xacro)
@@ -4,5 +4,5 @@
     <parent link="chassis"/>
     <child link="lidar"/>
-    <origin xyz= "${chassis_length/2 + lidar_length/2} 0 0" rpy="0 0 0"/>
+    <origin xyz= "${chassis_radius + lidar_length/2} 0 0" rpy="0 0 0"/>
   </joint>
   <link name="lidar">

File: description/property_macro.xacro (robot description, xacro)
@@ -17,6 +17,5 @@
   </material>
   <xacro:property name="chassis_height" value="0.2"/>
-  <xacro:property name="chassis_length" value="0.6"/>
-  <xacro:property name="chassis_width" value="0.6"/>
+  <xacro:property name="chassis_radius" value="0.3"/>
   <xacro:property name="wheel_radius" value="0.1"/>
   <xacro:property name="wheel_width" value="0.05"/>

File: description/robot_core.xacro (robot description, xacro)
@@ -14,10 +14,10 @@
     <parent link="base_link"/>
     <child link="chassis"/>
-    <origin xyz="${chassis_length/2} 0 ${chassis_height/2 + wheel_radius}"/>
+    <origin xyz="0 0 ${chassis_height/2 + wheel_radius}"/>
   </joint>
   <link name="chassis">
     <visual>
       <geometry>
-        <box size="${chassis_length} ${chassis_width} ${chassis_height}"/>
+        <cylinder radius="${chassis_radius}" length="${chassis_height}"/>
       </geometry>
       <material name="white"/>
@@ -25,8 +25,8 @@
     <collision>
       <geometry>
-        <box size="${chassis_length} ${chassis_width} ${chassis_height}"/>
+        <cylinder radius="${chassis_radius}" length="${chassis_height}"/>
       </geometry>
     </collision>
-    <xacro:inertial_box mass="0.7" x="${chassis_length}" y="${chassis_width}" z="${chassis_height}"/>
+    <xacro:inertial_cylinder mass="0.7" radius="${chassis_radius}" length="${chassis_height}"/>
   </link>
   <gazebo reference="chassis">
@@ -37,5 +37,5 @@
     <parent link="base_link"/>
     <child link="left_wheel"/>
-    <origin xyz="${chassis_length/3} ${chassis_width/2} ${wheel_radius}"/>
+    <origin xyz="0 ${chassis_radius} ${wheel_radius}"/>
     <axis xyz="0 1 0"/>
   </joint>
@@ -63,5 +63,5 @@
     <parent link="base_link"/>
     <child link="right_wheel"/>
-    <origin xyz="${chassis_length/3} ${-chassis_width/2} ${wheel_radius}"/>
+    <origin xyz="0 ${-chassis_radius} ${wheel_radius}"/>
     <axis xyz="0 1 0"/>
   </joint>
@@ -85,11 +85,11 @@
     <material>Gazebo/Blue</material>
   </gazebo>
-  <!-- CASTER WHEEL -->
-  <joint name="caster_wheel_joint" type="fixed">
+  <!-- CASTER WHEEL FRONT-->
+  <joint name="caster_wheel_front_joint" type="fixed">
     <parent link="base_link"/>
-    <child link="caster_wheel"/>
-    <origin xyz="${3*chassis_length/4} 0 ${wheel_radius}"/>
+    <child link="caster_wheel_front"/>
+    <origin xyz="${2*chassis_radius/3} 0 ${wheel_radius}"/>
   </joint>
-  <link name="caster_wheel">
+  <link name="caster_wheel_front">
     <visual>
       <geometry>
@@ -105,5 +105,30 @@
     <xacro:inertial_sphere mass="0.1" radius="${wheel_radius}"/>
   </link>
-  <gazebo reference="caster_wheel">
+  <gazebo reference="caster_wheel_front">
+    <material>Gazebo/Yellow</material>
+    <mu1 value="0.000"/>
+    <mu2 value="0.000"/>
+  </gazebo>
+  <!-- CASTER WHEEL BACK-->
+  <joint name="caster_wheel_back_joint" type="fixed">
+    <parent link="base_link"/>
+    <child link="caster_wheel_back"/>
+    <origin xyz="${-2*chassis_radius/3} 0 ${wheel_radius}"/>
+  </joint>
+  <link name="caster_wheel_back">
+    <visual>
+      <geometry>
+        <sphere radius="${wheel_radius}"/>
+      </geometry>
+      <material name="sunshine"/>
+    </visual>
+    <collision>
+      <geometry>
+        <sphere radius="${wheel_radius}"/>
+      </geometry>
+    </collision>
+    <xacro:inertial_sphere mass="0.1" radius="${wheel_radius}"/>
+  </link>
+  <gazebo reference="caster_wheel_back">
     <material>Gazebo/Yellow</material>
     <mu1 value="0.000"/>

Commit message: Fixded the vicious cycle: face left but blocked -> try to face north -> left not blocked anymore -> try to face left -> face left but blocked

File: description/lidar.xacro (robot description, xacro)
@@ -4,5 +4,5 @@
     <parent link="chassis"/>
     <child link="lidar"/>
-    <origin xyz= "${chassis_radius + lidar_length/2} 0 0" rpy="0 0 0"/>
+    <origin xyz= "${chassis_radius - lidar_length/2} 0 0" rpy="0 0 0"/>
   </joint>
   <link name="lidar">
